File: kicad/USB.kicad_sch (KiCad schematic)
At the start: 35 parts, among them J1 USB_B, J3 Conn_02x03_Counter_Clockwise, J4 USB_A_Stacked, U3 USB2514B_Bi, U4 24LC02, Y2 24Mhz

Commit message: continued work on fader pcb and redid all references more logicly
Parts:
- removed C19: 100n, Capacitor_SMD:C_0603_1608Metric_Pad1.08x0.95mm_HandSolder, symbol Device:C
- added C122: 100n, Capacitor_SMD:C_0603_1608Metric_Pad1.08x0.95mm_HandSolder, symbol Device:C
- U107: renamed from U4; footprint Package_SO:SOIC-8_3.9x4.9mm_P1.27mm -> Package_SO:SOP-8_3.9x4.9mm_P1.27mm
- renumbered C22 to C118, C16 to C119, C17 to C120, C18 to C121, C20 to C123, C21 to C124, C27 to C125, C28 to C126, C25 to C127, C26 to C128, C24 to C129, C23 to C130, D8 to D101, D9 to D102, D10 to D103, D2 to D104, D3 to D105, D4 to D106, D5 to D107, D6 to D108, D7 to D109, J3 to J104, J4 to J105, J1 to J106, R6 to R109, R7 to R110, R8 to R111, R12 to R112, R10 to R113, R11 to R114, R9 to R115, U3 to U106, Y2 to X201
Connections:
- net +3V3: now also C122.1
- net GND: now also C122.2
- no-connect marks 1 -> 2
