File: kicad/keypad.kicad_sch (KiCad schematic)
At the start: 77 parts, among them J10 Conn_01x05_Socket, J17 Conn_01x02_Socket, J23 Conn_01x04_Socket, J24 Conn_01x04_Socket, J25 Conn_01x04_Socket, J26 Conn_01x04_Socket, J27 Conn_01x04_Socket, J28 Conn_01x04_Socket, J29 Conn_01x04_Socket, J30 Conn_01x04_Socket, SW26 SW_SPST, SW27 SW_SPST, SW28 SW_SPST, SW29 SW_SPST, SW30 SW_SPST, SW31 SW_SPST, SW32 SW_SPST, SW33 SW_SPST, SW34 SW_SPST, SW35 SW_SPST, SW36 SW_SPST, SW37 SW_SPST, SW38 SW_SPST, SW39 SW_SPST, SW40 SW_SPST, SW41 SW_SPST, SW42 SW_SPST, SW43 SW_SPST, SW44 SW_SPST, SW45 SW_SPST, SW46 SW_SPST, SW47 SW_SPST, SW48 SW_SPST, SW49 SW_SPST, SW50 SW_SPST, SW51 SW_SPST, SW62 SW_SPST, SW63 SW_SPST, SW64 SW_SPST, SW65 SW_SPST, SW66 SW_SPST, SW67 SW_SPST, SW68 SW_SPST, SW69 SW_SPST, SW70 SW_SPST, SW71 SW_SPST, SW72 SW_SPST, SW73 SW_SPST, SW74 SW_SPST, SW75 SW_SPST, SW76 SW_SPST, SW77 SW_SPST, SW78 SW_SPST, SW79 SW_SPST, SW80 SW_SPST, SW81 SW_SPST, SW82 SW_SPST, SW83 SW_SPST, SW84 SW_SPST, U16 MTCH102, U18 DRV8210, U7 TCA8418

Commit message: continued work on fader pcb and redid all references more logicly
Parts:
- C61: now not fitted
- renumbered C33 to C501, C34 to C502, J17 to J502, J10 to J503, J23 to J504, J25 to J505, J24 to J506, J26 to J507, J27 to J508, J29 to J509, J28 to J510, J30 to J511, MF6 to MF501, R28 to R501, R29 to R502, R30 to R503, R31 to R504, R21 to R506, R20 to R507, SW62 to SW501, SW63 to SW502, SW64 to SW503, SW65 to SW504, SW66 to SW505, SW67 to SW506, SW68 to SW507, SW69 to SW508, SW70 to SW509, SW71 to SW510, SW72 to SW511, SW73 to SW512, SW74 to SW513, SW75 to SW514, SW76 to SW515, SW77 to SW516, SW78 to SW517, SW79 to SW518, SW80 to SW519, SW81 to SW520, SW82 to SW521, SW83 to SW522, SW84 to SW523, SW26 to SW524, SW27 to SW525, SW28 to SW526, SW29 to SW527, SW30 to SW528, SW31 to SW529, SW32 to SW530, SW33 to SW531, SW34 to SW532, SW35 to SW533, SW36 to SW534, SW37 to SW535, SW38 to SW536, SW39 to SW537, SW40 to SW538, SW41 to SW539, SW42 to SW540, SW43 to SW541, SW44 to SW542, SW45 to SW543, SW46 to SW544, SW47 to SW545, SW48 to SW546, SW49 to SW547, SW50 to SW548, SW51 to SW549, U7 to U501, U16 to U502
Connections:
- net +3V3: now also U501.21 (VCC)
- net INT-KEYP: now also U501.24 (~{INT})
- net SCL-KEYP: now also U501.23 (SCL); no longer U501.24 (~{INT})
- net SDA-KEYP: now also U501.22 (SDA); no longer U501.23 (SCL)
Other:
- note added: "J501"
- note added: "Put c508 on the motor terminal/fader directly use ceramic 100nf cap"
- note removed: "KEYPAD"
- moved on the sheet: R501, R502, R503, R504, R506, R507
