File: kicad/midi-controller.kicad_pcb (KiCad board)
At the start: 4 copper layers, 100 x 100 mm, 501 parts, among them J1 USB_B, J10 Conn_01x05_Socket, J11 AudioJack2, J12 AudioJack2, J13 AudioJack2, J14 Conn_01x06_Socket, J15 Conn_01x06_Socket, J16 Conn_01x06_Socket, J17 Conn_01x02_Socket, J18 Conn_01x05_Socket, J19 Conn_01x06_Socket, J2 Conn_02x03_Counter_Clockwise, J20 Conn_01x05_Socket, J21 Conn_01x06_Socket, J22 Conn_01x06_Socket, J23 Conn_01x04_Socket, J24 Conn_01x04_Socket, J25 Conn_01x04_Socket, J26 Conn_01x04_Socket, J27 Conn_01x04_Socket, J28 Conn_01x04_Socket, J29 Conn_01x04_Socket, J3 Conn_02x03_Counter_Clockwise, J30 Conn_01x04_Socket, J31 Conn_01x06_Socket, J32 Conn_01x06_Socket, J33 Conn_01x05_Socket, J34 Conn_01x05_Socket, J35 Conn_01x06_Socket, J36 Conn_01x06_Socket, J37 Conn_01x06_Socket, J38 Conn_01x06_Socket, J39 Conn_01x06_Socket, J4 USB_A_Stacked, J5 DIN-5_180degree, J6 DIN-5_180degree, J7 DIN-5_180degree, J8 Conn_01x07_Socket, J9 Conn_01x07_Socket, SW1 RotaryEncoder_Switch, SW10 RotaryEncoder_Switch, SW11 SW_SPST, SW12 SW_SPST, SW13 SW_SPST, SW14 SW_SPST, SW15 SW_SPST, SW16 SW_SPST, SW17 SW_SPST, SW18 SW_SPST, SW19 SW_SPST, SW2 RotaryEncoder_Switch, SW20 SW_SPST, SW21 SW_SPST, SW22 SW_SPST, SW23 SW_SPST, SW24 SW_SPST, SW25 SW_SPST, SW26 SW_SPST, SW27 SW_SPST, SW28 SW_SPST, SW29 SW_SPST, SW3 RotaryEncoder_Switch, SW30 SW_SPST, SW31 SW_SPST, SW32 SW_SPST, SW33 SW_SPST, SW34 SW_SPST, SW35 SW_SPST, SW36 SW_SPST, SW37 SW_SPST, SW38 SW_SPST, SW39 SW_SPST, SW4 RotaryEncoder_Switch, SW40 SW_SPST, SW41 SW_SPST, SW42 SW_SPST, SW43 SW_SPST, SW44 SW_SPST, SW45 SW_SPST, SW46 SW_SPST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

Commit message: update kicad files
Connections:
- U17 pad 12: M4B -> unconnected-(U17-LED6-Pad12)
- U17 pad 15: M3B -> unconnected-(U17-LED8-Pad15)
- U17 pad 17: M2B -> unconnected-(U17-LED10-Pad17)
- U17 pad 19: M1B -> unconnected-(U17-LED12-Pad19)
- U17 pad 21: M0B -> unconnected-(U17-LED14-Pad21)
Changed lines of the file:
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@@
 	(net 658 "unconnected-(U1-GPIO17-Pad28)")
 	(net 659 "unconnected-(U1-GPIO7-Pad9)")
+	(net 660 "unconnected-(U17-LED14-Pad21)")
+	(net 661 "unconnected-(U17-LED10-Pad17)")
+	(net 662 "unconnected-(U17-LED12-Pad19)")
+	(net 663 "unconnected-(U17-LED8-Pad15)")
+	(net 664 "unconnected-(U17-LED6-Pad12)")
 	(footprint "LED_SMD:LED_0603_1608Metric_Pad1.05x0.95mm_HandSolder"
 		(layer "F.Cu")
@@
 			(layers "F.Cu" "F.Paste" "F.Mask")
 			(roundrect_rratio 0.25)
-			(net 298 "M4B")
+			(net 664 "unconnected-(U17-LED6-Pad12)")
 			(pinfunction "LED6")
-			(pintype "output")
+			(pintype "output+no_connect")
 		)
 		(pad "13" smd roundrect
@@
 			(layers "F.Cu" "F.Paste" "F.Mask")
 			(roundrect_rratio 0.25)
-			(net 296 "M3B")
+			(net 663 "unconnected-(U17-LED8-Pad15)")
 			(pinfunction "LED8")
-			(pintype "output")
+			(pintype "output+no_connect")
 		)
 		(pad "16" smd roundrect
@@
 			(layers "F.Cu" "F.Paste" "F.Mask")
 			(roundrect_rratio 0.25)
-			(net 291 "M2B")
+			(net 661 "unconnected-(U17-LED10-Pad17)")
 			(pinfunction "LED10")
-			(pintype "output")
+			(pintype "output+no_connect")
 		)
 		(pad "18" smd roundrect
@@
 			(layers "F.Cu" "F.Paste" "F.Mask")
 			(roundrect_rratio 0.25)
-			(net 294 "M1B")
+			(net 662 "unconnected-(U17-LED12-Pad19)")
 			(pinfunction "LED12")
-			(pintype "output")
+			(pintype "output+no_connect")
 		)
 		(pad "20" smd roundrect
@@
 			(layers "F.Cu" "F.Paste" "F.Mask")
 			(roundrect_rratio 0.25)
-			(net 286 "M0B")
+			(net 660 "unconnected-(U17-LED14-Pad21)")
 			(pinfunction "LED14")
-			(pintype "output")
+			(pintype "output+no_connect")
 		)
 		(pad "22" smd roundrect

Commit message: continued work on fader pcb and redid all references more logicly
Parts:
- removed C19: 100n, Capacitor_SMD:C_0603_1608Metric_Pad1.08x0.95mm_HandSolder
- removed J22, J35, J36, J37, J38: Conn_01x06_Socket, Connector_JST:JST_XH_B6B-XH-A_1x06_P2.50mm_Vertical
- removed J33, J34: Conn_01x05_Socket, Connector_JST:JST_XH_B5B-XH-A_1x05_P2.50mm_Vertical
- removed JP2: SolderJumper_2_Open, Jumper:SolderJumper-2_P1.3mm_Open_RoundedPad1.0x1.5mm
- removed R46: 2K5, Resistor_SMD:R_0603_1608Metric_Pad0.98x0.95mm_HandSolder
- removed U10: MCP23S17_SO, Package_SO:SOIC-28W_7.5x17.9mm_P1.27mm
- removed U18, U19, U20, U21, U22: DRV8210, personal:SOT-6
- added C122: 100n, Capacitor_SMD:C_0603_1608Metric_Pad1.08x0.95mm_HandSolder, F.Cu at (132.1, 115.5)
- added C303: 100n, Capacitor_SMD:C_0603_1608Metric_Pad1.08x0.95mm_HandSolder, F.Cu at (48.5, 369.8)
- added C304: 100n, Capacitor_SMD:C_0603_1608Metric_Pad1.08x0.95mm_HandSolder, F.Cu at (48.5, 372.3)
- added C305: 1u, Capacitor_SMD:C_0603_1608Metric_Pad1.08x0.95mm_HandSolder, F.Cu at (48.5, 374.8)
- added C306: 100n, Capacitor_SMD:C_0603_1608Metric_Pad1.08x0.95mm_HandSolder, F.Cu at (48.5, 377.3)
- added C307: 100n, Capacitor_SMD:C_0603_1608Metric_Pad1.08x0.95mm_HandSolder, F.Cu at (48.5, 379.8)
- added C308: 100n, Capacitor_SMD:C_0603_1608Metric_Pad1.08x0.95mm_HandSolder, F.Cu at (48.5, 382.4)
- added C309: 100n, Capacitor_SMD:C_0603_1608Metric_Pad1.08x0.95mm_HandSolder, F.Cu at (48.5, 384.9)
- added C310: 100n, Capacitor_SMD:C_0603_1608Metric_Pad1.08x0.95mm_HandSolder, F.Cu at (48.5, 387.4)
- added C311: 100n, Capacitor_SMD:C_0603_1608Metric_Pad1.08x0.95mm_HandSolder, F.Cu at (48.5, 389.9)
- added C312: 1u, Capacitor_SMD:C_0603_1608Metric_Pad1.08x0.95mm_HandSolder, F.Cu at (48.5, 392.4)
- added C415: 100n, Capacitor_SMD:C_0603_1608Metric_Pad1.08x0.95mm_HandSolder, F.Cu at (61.6, 384.9)
- added C425: 100n, Capacitor_SMD:C_0603_1608Metric_Pad1.08x0.95mm_HandSolder, F.Cu at (66.0, 377.3)
- added R301: 1K, Resistor_SMD:R_0603_1608Metric_Pad0.98x0.95mm_HandSolder, F.Cu at (70.3, 392.4)
- added R302: NFIT, Resistor_SMD:R_0603_1608Metric_Pad0.98x0.95mm_HandSolder, F.Cu at (74.7, 362.3)
- added R303: 1K, Resistor_SMD:R_0603_1608Metric_Pad0.98x0.95mm_HandSolder, F.Cu at (74.7, 364.8)
- added R304: 10K, Resistor_SMD:R_0603_1608Metric_Pad0.98x0.95mm_HandSolder, F.Cu at (74.7, 367.3)
- added R321: 80K, Resistor_SMD:R_0603_1608Metric_Pad0.98x0.95mm_HandSolder, F.Cu at (79.0, 377.3)
- added R322: 80K, Resistor_SMD:R_0603_1608Metric_Pad0.98x0.95mm_HandSolder, F.Cu at (79.0, 379.8)
- added R323: 80K, Resistor_SMD:R_0603_1608Metric_Pad0.98x0.95mm_HandSolder, F.Cu at (79.0, 382.4)
- added R324: 80K, Resistor_SMD:R_0603_1608Metric_Pad0.98x0.95mm_HandSolder, F.Cu at (79.0, 384.9)
- added R325: 80K, Resistor_SMD:R_0603_1608Metric_Pad0.98x0.95mm_HandSolder, F.Cu at (79.0, 387.4)
- added R403: 2K5, Resistor_SMD:R_0603_1608Metric_Pad0.98x0.95mm_HandSolder, F.Cu at (83.3, 362.3)
- added U301: RP2040, Package_DFN_QFN:QFN-56-1EP_7x7mm_P0.4mm_EP3.2x3.2mm, F.Cu at (230.3, 414.8)
- added U302: AT25SF081-SSHD-X, Package_SO:SOIC-8_3.9x4.9mm_P1.27mm, F.Cu at (223.2, 382.9)
- added U308: DRV8871DDA, Package_SO:Texas_HTSOP-8-1EP_3.9x4.9mm_P1.27mm_EP2.95x4.9mm_Mask2.4x3.1mm_ThermalVias, F.Cu at (109.7, 364.4)
- added U309: DRV8871DDA, Package_SO:Texas_HTSOP-8-1EP_3.9x4.9mm_P1.27mm_EP2.95x4.9mm_Mask2.4x3.1mm_ThermalVias, F.Cu at (109.7, 371.0)
- added U310: DRV8871DDA, Package_SO:Texas_HTSOP-8-1EP_3.9x4.9mm_P1.27mm_EP2.95x4.9mm_Mask2.4x3.1mm_ThermalVias, F.Cu at (109.7, 377.7)
- added U311: DRV8871DDA, Package_SO:Texas_HTSOP-8-1EP_3.9x4.9mm_P1.27mm_EP2.95x4.9mm_Mask2.4x3.1mm_ThermalVias, F.Cu at (109.7, 384.3)
- added U312: DRV8871DDA, Package_SO:Texas_HTSOP-8-1EP_3.9x4.9mm_P1.27mm_EP2.95x4.9mm_Mask2.4x3.1mm_ThermalVias, F.Cu at (109.7, 390.9)
- added X301: 12Mhz, Crystal:Crystal_SMD_HC49-SD, F.Cu at (66.6, 411.7)
- C336: renamed from C37; value 1u -> 2u2
- C338: renamed from C80; value 100n -> 27p
- C339: renamed from C90; value 100n -> 27p
- J207: renamed from J13; value AudioJack2 -> AudioJack3
- J301: renamed from J16; value Conn_01x06_Socket -> Conn_02x03_Counter_Clockwise; footprint Connector_JST:JST_XH_B6B-XH-A_1x06_P2.50mm_Vertical -> Connector_PinHeader_2.54mm:PinHeader_2x03_P2.54mm_Vertical
- U107: renamed from U4; footprint Package_SO:SOIC-8_3.9x4.9mm_P1.27mm -> Package_SO:SOP-8_3.9x4.9mm_P1.27mm
- U403: renamed from U13; footprint Package_SO:SOIC-18W_7.5x11.6mm_P1.27mm -> Package_SO:SOIC-28W_7.5x17.9mm_P1.27mm
- moved U303 144.9 mm to (63.7, 418.1)
- moved U305 144.2 mm to (244.8, 420.4)
- moved J205 138.4 mm to (61.6, 403.8)
- moved J206 138.4 mm to (66.2, 403.8)
- moved J207 138.4 mm to (70.8, 403.8)
- moved U407 135.6 mm to (231.7, 382.9)
- moved U408 135.6 mm to (231.7, 389.4)
- moved U411 135.2 mm to (240.2, 382.9)
- moved U412 135.2 mm to (240.2, 389.4)
- moved U413 135.2 mm to (240.2, 396.0)
- moved C501 133.3 mm to (226.9, 408.0)
- moved C502 133.3 mm to (229.4, 408.0)
- moved R501 133.3 mm to (231.9, 408.0)
- moved R502 133.3 mm to (234.4, 408.0)
- moved R503 133.3 mm to (236.9, 408.0)
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- renumbered C8 to C101, C9 to C102, C10 to C103, C11 to C104, C12 to C105, C13 to C106, C14 to C107, C5 to C108, C7 to C109, C6 to C110, C3 to C111, C4 to C112, C1 to C113, C2 to C114, C15 to C115, C32 to C116, C93 to C117, C22 to C118, C16 to C119, C17 to C120, C18 to C121, C20 to C123, C21 to C124, C27 to C125, C28 to C126, C25 to C127, C26 to C128, C24 to C129, C23 to C130, C31 to C201, C29 to C202, C30 to C203, C72 to C301, C35 to C313, C36 to C314, C47 to C315, C48 to C316, C70 to C317, C71 to C318, C51 to C319, C52 to C320, C53 to C321, C54 to C322, C55 to C323, C56 to C324, C57 to C325, C58 to C326, C59 to C327, C60 to C328, C45 to C334, C46 to C335, C38 to C337, C66 to C401, C39 to C402, C40 to C403, C41 to C404, C42 to C405, C43 to C406, C44 to C407, C73 to C408, C74 to C409, C75 to C410, C76 to C411, C77 to C412, C78 to C413, C79 to C414, C81 to C416, C82 to C417, C83 to C418, C84 to C419, C85 to C420, C86 to C421, C87 to C422, C88 to C423, C89 to C424, C91 to C426, C92 to C427, C33 to C501, C34 to C502, C49 to C503, C50 to C504, C67 to C506, C68 to C507, D8 to D101, D9 to D102, D10 to D103, D2 to D104, D3 to D105, D4 to D106, D5 to D107, D6 to D108, D7 to D109, D1 to D201, D11 to D4000, D12 to D4001, D13 to D4002, D14 to D4003, D15 to D4004, D16 to D4005, D17 to D4006, D18 to D4007, D19 to D4008, D20 to D4009, D21 to D4010, D22 to D4011, D23 to D4012, D24 to D4013, D25 to D4014, D26 to D4015, D27 to D4016, D28 to D4017, D29 to D4018, D30 to D4019, D31 to D4020, D32 to D4021, D33 to D4022, D34 to D4023, D35 to D4024, D36 to D4025, D37 to D4026, D38 to D4027, D39 to D4028, D40 to D4029, D41 to D4030, D42 to D4031, D43 to D4032, D44 to D4033, D45 to D4034, D46 to D4035, D47 to D4036, D48 to D4037, D49 to D4038, D50 to D4039, D51 to D4040, D52 to D4041, D53 to D4042, D54 to D4043, D55 to D4044, D56 to D4045, D57 to D4046, D58 to D4047, D59 to D4048, D60 to D4049, D61 to D4050, D62 to D4051, D63 to D4052, D64 to D4053, D65 to D4054, D66 to D4055, D67 to D4056, D68 to D4057, D69 to D4058, D70 to D4059, D71 to D4060, D72 to D4061, D73 to D4062, D74 to D4063, D75 to D4064, D76 to D4065, D77 to D4066, D78 to D4067, D79 to D4068, D80 to D4069, D81 to D4070, D82 to D4071, D83 to D4072, D84 to D4073, D85 to D4074, D86 to D4075, D87 to D4076, D88 to D4077, D89 to D4078, D90 to D4079, D91 to D4080, D92 to D4081, D93 to D4082, D94 to D4083, D95 to D4084, D96 to D4085, D97 to D4086, D98 to D4087, D99 to D4088, D100 to D4089, D101 to D4090, D102 to D4091, D103 to D4092, D104 to D4093, D105 to D4094, D106 to D4095, D107 to D4096, D108 to D4097, D109 to D4098, D110 to D4099, D111 to D4100, D112 to D4101, D113 to D4102, D114 to D4103, D115 to D4104, D116 to D4105, D117 to D4106, D118 to D4107, D119 to D4108, D120 to D4109, D121 to D4110, D122 to D4111, D123 to D4112, D124 to D4113, D125 to D4114, D126 to D4115, D127 to D4116, D128 to D4117, D129 to D4118, D130 to D4119, D131 to D4120, D132 to D4121, D133 to D4122, D134 to D4123, D135 to D4124, D136 to D4125, D137 to D4126, D138 to D4127, D139 to D4128, D140 to D4129, D141 to D4130, D142 to D4131, D143 to D4132, D144 to D4133, D145 to D4134, D146 to D4135, D147 to D4136, D148 to D4137, D149 to D4138, D150 to D4139, D151 to D4140, D152 to D4141, D153 to D4142, D154 to D4143, D155 to D4144, D156 to D4145, D157 to D4146, D158 to D4147, D159 to D4148, D160 to D4149, D161 to D4150, D162 to D4151, D163 to D4152, D164 to D4153, D165 to D4154, D166 to D4155, D167 to D4156, D168 to D4157, D169 to D4158, D170 to D4159, D171 to D4160, D173 to D4161, D175 to D4162, D177 to D4163, D179 to D4164, D172 to D4165, D174 to D4166, D176 to D4167, D178 to D4168, D180 to D4169, DS1 to DS301, DS2 to DS302, DS3 to DS303, DS4 to DS304, DS5 to DS305, DS6 to DS501, FB1 to FB201, FB2 to FB202, FB3 to FB203, FB4 to FB204, FB5 to FB205, FB6 to FB206, J2 to J101, J8 to J102, J39 to J103, J3 to J104, J4 to J105, J1 to J106, J9 to J201, J5 to J202, J6 to J203, J7 to J204, J11 to J205, J12 to J206, J15 to J302, J14 to J303, J19 to J307, J21 to J308, J18 to J309, J20 to J310, J31 to J311, J32 to J312, J17 to J502, J10 to J503, J23 to J504, J25 to J505, J24 to J506, J26 to J507, J27 to J508, J29 to J509, J28 to J510, J30 to J511, JP1 to JP101, MF1 to MF301, MF2 to MF302, MF3 to MF303, MF4 to MF304, MF5 to MF305, MF6 to MF501, R23 to R101, R3 to R102, R4 to R103, R2 to R104, R1 to R105, R32 to R106, R5 to R107, R19 to R108, R6 to R109, R7 to R110, R8 to R111, R12 to R112, R10 to R113, R11 to R114, R9 to R115, R18 to R201, R14 to R202, R15 to R203, R16 to R204, R17 to R205, R13 to R206, R36 to R305, R37 to R306, R38 to R307, R39 to R308, R40 to R309, R45 to R310, R44 to R311, R43 to R312, R42 to R313, R41 to R314, R22 to R315, R24 to R316, R25 to R317, R26 to R318, R27 to R319, R33 to R320, R34 to R401, R35 to R402, R47 to R404, R48 to R405, R49 to R406, R50 to R407, R51 to R408, R52 to R409, R53 to R410, R28 to R501, R29 to R502, R30 to R503, R31 to R504, R21 to R506, R20 to R507, RV1 to RV301, SW11 to SW300, SW12 to SW301, SW13 to SW302, SW14 to SW303, SW15 to SW304, SW1 to SW400, SW2 to SW401, SW3 to SW402, SW4 to SW403, SW5 to SW404, SW6 to SW405, SW7 to SW406, SW8 to SW407, SW9 to SW408, SW10 to SW409, SW16 to SW410, SW17 to SW411, SW18 to SW412, SW19 to SW413, SW20 to SW414, SW21 to SW415, SW22 to SW416, SW23 to SW417, SW24 to SW418, SW25 to SW419, SW62 to SW501, SW63 to SW502, SW64 to SW503, SW65 to SW504, SW66 to SW505, SW67 to SW506, SW68 to SW507, SW69 to SW508, SW70 to SW509, SW71 to SW510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
Connections:
- C338 pad 1: +E3V3 -> FGND
- C338 pad 2: EGND -> /Fader-bank/FXIN
- C339 pad 1: +E3V3 -> FGND
- C339 pad 2: EGND -> Net-(C339-Pad2)
- C418 pad 1: +E3V3 -> Net-(U419-VCC)
- C419 pad 1: +E3V3 -> Net-(U419-VCC)
- C426 pad 2: EGND -> Net-(C426-Pad2)
- C427 pad 2: EGND -> Net-(C426-Pad2)
- D4096 pad 2: +E3V3 -> Net-(D4096-A)
- D4097 pad 2: +E3V3 -> Net-(D4096-A)
- D4098 pad 2: +E3V3 -> Net-(D4096-A)
- D4099 pad 2: +E3V3 -> Net-(D4096-A)
- D4100 pad 2: +E3V3 -> Net-(D4096-A)
- D4101 pad 2: +E3V3 -> Net-(D4096-A)
- D4102 pad 2: +E3V3 -> Net-(D4096-A)
- D4103 pad 2: +E3V3 -> Net-(D4096-A)
- D4104 pad 2: +E3V3 -> Net-(D4096-A)
- D4105 pad 2: +E3V3 -> Net-(D4096-A)
- D4106 pad 2: +E3V3 -> Net-(D4096-A)
- D4107 pad 2: +E3V3 -> Net-(D4096-A)
- D4108 pad 2: +E3V3 -> Net-(D4096-A)
- D4109 pad 2: +E3V3 -> Net-(D4096-A)
- D4110 pad 2: +E3V3 -> Net-(D4096-A)
- D4111 pad 2: +E3V3 -> Net-(D4096-A)
- D4166 pad 2: +E3V3 -> Net-(D4096-A)
- J106 pad 5: Net-(J1-Shield) -> unconnected-(J106-Shield-Pad5)
- J207 pad 1: unconnected-(J13-S-Pad1) -> (no net)
- J207 pad 2: M-FPEDAL1 -> (no net)
- J301 pad 1: FWINT -> +F3V3
- J301 pad 2: FWCS -> FGND
- J301 pad 3: FSPI1SCL -> F_BOOTSEL
- J301 pad 4: FSPI1MOSI -> F_RESET_RP2
- J301 pad 5: FSPI1MISO -> F_SWDIO
- J301 pad 6: FGND -> F_SWCLK
- J307 pad 1: Net-(J19-Pin_1) -> INT_U11
- J307 pad 2: Net-(J19-Pin_2) -> CS_U11
- J307 pad 3: Net-(J19-Pin_3) -> INT_U12
- J307 pad 4: Net-(J19-Pin_4) -> CS_U12
- J307 pad 5: Net-(J19-Pin_5) -> INT_U13
- J307 pad 6: Net-(J19-Pin_6) -> CS_U13
- J310 pad 3: SPI0SCK-ENC -> SPI1SCK-ENC
- J310 pad 4: SPI0MOSI-ENC -> SPI1MOSI-ENC
- J310 pad 5: SPI0MISO-ENC -> SPI1MISO-ENC
- R408 pad 1: unconnected-(R51-Pad1) -> EGND
- U101 pad 2: SPI0MISO -> unconnected-(U101-GPIO0-Pad2)
- U101 pad 3: SPI0DC -> unconnected-(U101-GPIO1-Pad3)
- U101 pad 4: SPI0SCK -> unconnected-(U101-GPIO2-Pad4)
- U101 pad 5: SPI0MOSI -> unconnected-(U101-GPIO3-Pad5)
- U101 pad 6: SDA -> unconnected-(U101-GPIO4-Pad6)
- U101 pad 7: SCL -> unconnected-(U101-GPIO5-Pad7)
- U306 pad 1: Net-(JP2-B) -> FGND
- U306 pad 12: unconnected-(U17-LED6-Pad12) -> M4B
- U306 pad 15: unconnected-(U17-LED8-Pad15) -> M3B
- U306 pad 17: unconnected-(U17-LED10-Pad17) -> M2B
- U306 pad 19: unconnected-(U17-LED12-Pad19) -> M1B
- U306 pad 2: unconnected-(U17-A1-Pad2) -> FGND
- U306 pad 21: unconnected-(U17-LED14-Pad21) -> M0B
- U306 pad 24: unconnected-(U17-A5-Pad24) -> FGND
- U306 pad 3: unconnected-(U17-A2-Pad3) -> FGND
- U306 pad 4: unconnected-(U17-A3-Pad4) -> FGND
- U306 pad 5: unconnected-(U17-A4-Pad5) -> FGND
- U401 pad 12: SPI0SCK-ENC -> SPI1SCK-ENC
- U401 pad 13: SPI0MOSI-ENC -> SPI1MOSI-ENC
- U401 pad 14: SPI0MISO-ENC -> SPI1MISO-ENC
- U402 pad 12: SPI0SCK-ENC -> SPI1SCK-ENC
- U402 pad 13: SPI0MOSI-ENC -> SPI1MOSI-ENC
- U402 pad 14: SPI0MISO-ENC -> SPI1MISO-ENC
- U403 pad 1: SPI0SCK-ENC -> Net-(U403-GPB0)
- U403 pad 10: Net-(U13-GP0) -> EGND
- U403 pad 11: Net-(U13-GP1) -> CS_U13-ENC
- U403 pad 12: Net-(U13-GP2) -> SPI1SCK-ENC
- U403 pad 13: B09 -> SPI1MOSI-ENC
- U403 pad 14: B14 -> SPI1MISO-ENC
- U403 pad 15: Net-(U13-GP5) -> EGND
- U403 pad 16: Net-(U13-GP6) -> EGND
- U403 pad 17: Net-(U13-GP7) -> EGND
- U403 pad 18: +E3V3 -> ~{ERST}
- U403 pad 2: SPI0MOSI-ENC -> Net-(U403-GPB1)
- U403 pad 3: SPI0MISO-ENC -> Net-(U403-GPB2)
- U403 pad 4: EGND -> B09
- U403 pad 5: EGND -> B14
- U403 pad 6: ~{ERST} -> Net-(U403-GPB5)
- U403 pad 7: CS_U13-ENC -> Net-(U403-GPB6)
- U403 pad 8: INT_U13-ENC -> Net-(U403-GPB7)
- U403 pad 9: EGND -> +E3V3
- U408 pad 5: Net-(U13-GP2) -> Net-(U403-GPB2)
- U408 pad 6: Net-(U13-GP1) -> Net-(U403-GPB1)
- U408 pad 7: Net-(U13-GP0) -> Net-(U403-GPB0)
- U413 pad 5: Net-(U13-GP7) -> Net-(U403-GPB7)
- U413 pad 6: Net-(U13-GP6) -> Net-(U403-GPB6)
- U413 pad 7: Net-(U13-GP5) -> Net-(U403-GPB5)
- U419 pad 24: +E3V3 -> Net-(U419-VCC)
- U420 pad 1: EGND -> unconnected-(U420-GND-Pad1)
- U501 pad 21: unconnected-(U7-VCC-Pad21) -> +3V3
- U501 pad 22: unconnected-(U7-SDA-Pad22) -> SDA-KEYP
- U501 pad 23: SDA-KEYP -> SCL-KEYP
- U501 pad 24: SCL-KEYP -> INT-KEYP
Routing:
- net (no net): track 22.0 -> 0.00 mm, vias 13 -> 0
- net unconnected-(U101-GPIO0-Pad2): track 0.00 -> 16.2 mm
- net SPI0MISO: track 16.2 -> 0.00 mm
- net unconnected-(U101-GPIO1-Pad3): track 0.00 -> 15.5 mm
- net SPI0DC: track 15.5 -> 0.00 mm
- net unconnected-(U101-GPIO2-Pad4): track 0.00 -> 14.9 mm
- net SPI0SCK: track 14.9 -> 0.00 mm
- net unconnected-(U101-GPIO3-Pad5): track 0.00 -> 14.2 mm
- net SPI0MOSI: track 14.2 -> 0.00 mm
- net unconnected-(U101-GPIO4-Pad6): track 0.00 -> 13.5 mm
- net SDA: track 13.5 -> 0.00 mm
- net unconnected-(U101-GPIO5-Pad7): track 0.00 -> 12.9 mm
- net SCL: track 12.9 -> 0.00 mm
- net GND: track 22.3 -> 29.6 mm, vias 27 -> 30
- net VBUS_IN: track 14.1 -> 17.0 mm
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- added copper zone on In1.Cu, net GND
- removed copper zone on In1.Cu, net EGND
- removed copper zone on In1.Cu, net FGND
