File: kicad/faders.kicad_sch (KiCad schematic)
At the start: 140 parts, among them J301 Conn_02x03_Counter_Clockwise, J302 Conn_01x06_Socket, J303 Conn_01x06_Socket, J307 Conn_01x06_Socket, J308 Conn_01x06_Socket, J309 Conn_01x05_Socket, J310 Conn_01x05_Socket, J311 Conn_01x06_Socket, J312 Conn_01x06_Socket, SW300 SW_SPST, SW301 SW_SPST, SW302 SW_SPST, SW303 SW_SPST, SW304 SW_SPST, SW400 RotaryEncoder_Switch, SW401 RotaryEncoder_Switch, SW402 RotaryEncoder_Switch, SW403 RotaryEncoder_Switch, SW404 RotaryEncoder_Switch, SW405 RotaryEncoder_Switch, SW406 RotaryEncoder_Switch, SW407 RotaryEncoder_Switch, SW408 RotaryEncoder_Switch, SW409 RotaryEncoder_Switch, SW410 SW_SPST, SW411 SW_SPST, SW412 SW_SPST, SW413 SW_SPST, SW414 SW_SPST, SW415 SW_SPST, SW416 SW_SPST, SW417 SW_SPST, SW418 SW_SPST, SW419 SW_SPST, U301 RP2040, U302 AT25SF081-SSHD-X, U303 MTCH105, U304 MCP3008, U305 LM4040D33, U306 PCA9635, U307 MCP23S17_SO, U308 DRV8871DDA, U309 DRV8871DDA, U310 DRV8871DDA, U311 DRV8871DDA, U312 DRV8871DDA, U401 MCP23S17_SO, U402 MCP23S17_SO, U403 MCP23S17_SO, U404 LS30, U405 LS30, U406 LS30, U407 LS30, U408 LS30, U409 LS30, U410 LS30, U411 LS30, U412 LS30, U413 LS30, X301 12Mhz

Commit message: some more progress on the fader pcb and small changes to schematic
Connections:
- net FSPI1SCK is gone; now on net FSPI1SCL: DS301.4 (SCK), DS302.4 (SCK), DS303.4 (SCK), DS304.4 (SCK), DS305.4 (SCK)
- net E8S: now also SW408.S1; no longer SW408.S2
- net E9S: now also SW409.S1; no longer SW409.S2
- net EGND: now also SW408.S2, SW409.S2; no longer SW408.S1, SW409.S1
Other:
- note added: "place c305 close to pin 44 of rp2040"
- note added: "place c312 close to pin 45 of rp2040"
- note removed: "place c5 close to pin 45 of rp2040"
- note removed: "place c8 close to pin 44 of rp2040"
Changed lines of the file:
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@@
 	(wire
 		(pts
-			(xy 209.55 87.63) (xy 209.55 91.44)
+			(xy 205.74 92.71) (xy 205.74 93.98)
 		)
 		(stroke
@@
 	(wire
 		(pts
-			(xy 260.35 87.63) (xy 260.35 91.44)
-		)
-		(stroke
-			(width 0)
-			(type default)
-		)
-	)
-	(wire
-		(pts
 			(xy 234.95 248.92) (xy 237.49 248.92)
 		)
@@
 	(wire
 		(pts
-			(xy 199.39 87.63) (xy 209.55 87.63)
+			(xy 199.39 92.71) (xy 205.74 92.71)
 		)
 		(stroke
@@
 	(wire
 		(pts
+			(xy 256.54 92.71) (xy 250.19 92.71)
+		)
+		(stroke
+			(width 0)
+			(type default)
+		)
+	)
+	(wire
+		(pts
 			(xy 407.67 262.89) (xy 410.21 262.89)
 		)
@@
 	(wire
 		(pts
+			(xy 256.54 93.98) (xy 256.54 92.71)
+		)
+		(stroke
+			(width 0)
+			(type default)
+		)
+	)
+	(wire
+		(pts
 			(xy 31.75 49.53) (xy 31.75 48.26)
 		)
@@
 	(wire
 		(pts
-			(xy 250.19 92.71) (xy 251.46 92.71)
+			(xy 250.19 87.63) (xy 251.46 87.63)
 		)
 		(stroke
@@
 	(wire
 		(pts
+			(xy 199.39 87.63) (xy 200.66 87.63)
+		)
+		(stroke
+			(width 0)
+			(type default)
+		)
+	)
+	(wire
+		(pts
 			(xy 363.22 187.96) (xy 363.22 189.23)
 		)
@@
 	(wire
 		(pts
-			(xy 199.39 92.71) (xy 200.66 92.71)
-		)
-		(stroke
-			(width 0)
-			(type default)
-		)
-	)
-	(wire
-		(pts
 			(xy 297.18 214.63) (xy 297.18 215.9)
 		)
@@
 	(wire
 		(pts
-			(xy 250.19 87.63) (xy 260.35 87.63)
-		)
-		(stroke
-			(width 0)
-			(type default)
-		)
-	)
-	(wire
-		(pts
 			(xy 200.66 384.81) (xy 201.93 384.81)
 		)
@@
 		)
 	)
-	(text "place c8\nclose to\npin 44\nof rp2040"
+	(text "place c305\nclose to\npin 44\nof rp2040"
 		(exclude_from_sim no)
 		(at 381 180.34 0)
@@
 		)
 	)
-	(text "place c5 close to\npin 45 of rp2040"
+	(text "place c312 close to\npin 45 of rp2040"
 		(exclude_from_sim no)
 		(at 345.44 189.23 0)
@@
 	(global_label "E8S"
 		(shape input)
-		(at 200.66 92.71 0)
+		(at 200.66 87.63 0)
 		(fields_autoplaced yes)
 		(effects
@@
 		)
 		(property "Intersheetrefs" "${INTERSHEET_REFS}"
-			(at 207.2132 92.71 0)
+			(at 207.2132 87.63 0)
 			(effects
 				(font
@@
 		)
 	)
-	(global_label "FSPI1SCK"
+	(global_label "FSPI1SCL"
 		(shape input)
 		(at 128.27 149.86 180)
@@
 		)
 	)
-	(global_label "FSPI1SCK"
+	(global_label "FSPI1SCL"
 		(shape input)
 		(at 26.67 149.86 180)
@@
 		)
 	)
-	(global_label "FSPI1SCK"
+	(global_label "FSPI1SCL"
 		(shape input)
 		(at 77.47 149.86 180)
@@
 		)
 	)
-	(global_label "FSPI1SCK"
+	(global_label "FSPI1SCL"
 		(shape input)
 		(at 229.87 149.86 180)
@@
 		)
 	)
-	(global_label "FSPI1SCK"
+	(global_label "FSPI1SCL"
 		(shape input)
 		(at 179.07 149.86 180)
@@
 	(global_label "E9S"
 		(shape input)
-		(at 251.46 92.71 0)
+		(at 251.46 87.63 0)
 		(fields_autoplaced yes)
 		(effects
@@
 		)
 		(property "Intersheetrefs" "${INTERSHEET_REFS}"
-			(at 258.0132 92.71 0)
+			(at 258.0132 87.63 0)
 			(effects
 				(font
@@
 	)
 	(symbol
-		(lib_id "power:GND")
-		(at 260.35 91.44 0)
-		(mirror y)
-		(unit 1)
-		(exclude_from_sim no)
-		(in_bom yes)
-		(on_board yes)
-		(dnp no)
-		(property "Reference" "#PWR086"
-			(at 260.35 97.79 0)
-			(effects
-				(font
-					(size 1.27 1.27)
-				)
-				(hide yes)
-			)
-		)
-		(property "Value" "EGND"
-			(at 260.35 95.25 0)
-			(effects
-				(font
-					(size 1.27 1.27)
-				)
-			)
-		)
-		(property "Footprint" ""
-			(at 260.35 91.44 0)
-			(effects
-				(font
-					(size 1.27 1.27)
-				)
-				(hide yes)
-			)
-		)
-		(property "Datasheet" ""
-			(at 260.35 91.44 0)
-			(effects
-				(font
-					(size 1.27 1.27)
-				)
-				(hide yes)
-			)
-		)
-		(property "Description" ""
-			(at 260.35 91.44 0)
-			(effects
-				(font
-					(size 1.27 1.27)
-				)
-				(hide yes)
-			)
-		)
-		(pin "1"
-		)
-		(instances
-			(project "faders"
-				(path "/077511d1-9e66-4142-bbad-77a69cc748a7"
-					(reference "#PWR086")
-					(unit 1)
-				)
-			)
-			(project "midi-controller"
-				(path "/2cba2024-755f-4534-8b6f-a95a551957b1/f0e0d697-e432-4b50-8287-c9353a450074"
-					(reference "#PWR0192")
-					(unit 1)
-				)
-			)
-		)
-	)
-	(symbol
 		(lib_id "Device:C")
 		(at 92.075 176.53 0)
@@
 	(symbol
 		(lib_id "power:GND")
+		(at 256.54 93.98 0)
+		(unit 1)
+		(exclude_from_sim no)
+		(in_bom yes)
+		(on_board yes)
+		(dnp no)
+		(property "Reference" "#PWR05001"
+			(at 256.54 100.33 0)
+			(effects
+				(font
+					(size 1.27 1.27)
+				)
+				(hide yes)
+			)
+		)
+		(property "Value" "EGND"
+			(at 256.54 97.79 0)
+			(effects
+				(font
+					(size 1.27 1.27)
+				)
+			)
+		)
+		(property "Footprint" ""
+			(at 256.54 93.98 0)
+			(effects
+				(font
+					(size 1.27 1.27)
+				)
+				(hide yes)
+			)
+		)
+		(property "Datasheet" ""
+			(at 256.54 93.98 0)
+			(effects
+				(font
+					(size 1.27 1.27)
+				)
+				(hide yes)
+			)
+		)
+		(property "Description" ""
+			(at 256.54 93.98 0)
+			(effects
+				(font
+					(size 1.27 1.27)
+				)
+				(hide yes)
+			)
+		)
+		(pin "1"
+		)
+		(instances
+			(project "faders"
+				(path "/077511d1-9e66-4142-bbad-77a69cc748a7"
+					(reference "#PWR05001")
+					(unit 1)
+				)
+			)
+		)
+	)
+	(symbol
+		(lib_id "power:GND")
 		(at 31.75 49.53 0)
 		(unit 1)
@@
 	(symbol
 		(lib_id "power:GND")
-		(at 209.55 91.44 0)
-		(mirror y)
+		(at 205.74 93.98 0)
 		(unit 1)
 		(exclude_from_sim no)
@@
 		(dnp no)
 		(property "Reference" "#PWR084"
-			(at 209.55 97.79 0)
+			(at 205.74 100.33 0)
 			(effects
 				(font
@@
 		)
 		(property "Value" "EGND"
-			(at 209.55 95.25 0)
+			(at 205.74 97.79 0)
 			(effects
 				(font
@@
 		)
 		(property "Footprint" ""
-			(at 209.55 91.44 0)
+			(at 205.74 93.98 0)
 			(effects
 				(font
@@
 		)
 		(property "Datasheet" ""
-			(at 209.55 91.44 0)
+			(at 205.74 93.98 0)
 			(effects
 				(font
@@
 		)
 		(property "Description" ""
-			(at 209.55 91.44 0)
+			(at 205.74 93.98 0)
 			(effects
 				(font
