File: kicad/faders.kicad_sch (KiCad schematic)
At the start: 140 parts, among them J301 Conn_02x03_Counter_Clockwise, J302 Conn_01x06_Socket, J303 Conn_01x06_Socket, J307 Conn_01x06_Socket, J308 Conn_01x06_Socket, J309 Conn_01x05_Socket, J310 Conn_01x05_Socket, J311 Conn_01x06_Socket, J312 Conn_01x06_Socket, SW300 SW_SPST, SW301 SW_SPST, SW302 SW_SPST, SW303 SW_SPST, SW304 SW_SPST, SW400 RotaryEncoder_Switch, SW401 RotaryEncoder_Switch, SW402 RotaryEncoder_Switch, SW403 RotaryEncoder_Switch, SW404 RotaryEncoder_Switch, SW405 RotaryEncoder_Switch, SW406 RotaryEncoder_Switch, SW407 RotaryEncoder_Switch, SW408 RotaryEncoder_Switch, SW409 RotaryEncoder_Switch, SW410 SW_SPST, SW411 SW_SPST, SW412 SW_SPST, SW413 SW_SPST, SW414 SW_SPST, SW415 SW_SPST, SW416 SW_SPST, SW417 SW_SPST, SW418 SW_SPST, SW419 SW_SPST, U301 RP2040, U302 AT25SF081-SSHD-X, U303 MTCH105, U304 MCP3008, U305 LM4040D33, U306 PCA9635, U307 MCP23S17_SO, U308 DRV8871DDA, U309 DRV8871DDA, U310 DRV8871DDA, U311 DRV8871DDA, U312 DRV8871DDA, U401 MCP23S17_SO, U402 MCP23S17_SO, U403 MCP23S17_SO, U404 LS30, U405 LS30, U406 LS30, U407 LS30, U408 LS30, U409 LS30, U410 LS30, U411 LS30, U412 LS30, U413 LS30, X301 12Mhz

Commit message: pushed unsaved kicad files. don't know what changed
Parts:
- added J313: Conn_01x06_Socket, Connector_JST:JST_XH_B6B-XH-A_1x06_P2.50mm_Vertical, symbol Connector:Conn_01x06_Socket
- added J314, J315: Conn_01x03_Socket, Connector_JST:JST_XH_B3B-XH-A_1x03_P2.50mm_Vertical, symbol Connector:Conn_01x03_Socket
- J309, J310: footprint Connector_JST:JST_XH_B5B-XH-A_1x05_P2.50mm_Vertical -> Connector_JST:JST_XH_B6B-XH-A_1x06_P2.50mm_Vertical; symbol Connector:Conn_01x05_Socket -> Connector:Conn_01x06_Socket
Connections:
- net +F3V3: now also J309.5 (Pin_5); no longer J309.4 (Pin_4)
- net BGND: now also SW300.1 (GND), SW301.1 (GND), SW302.1 (GND), SW303.1 (GND), SW304.1 (GND), J314.1 (Pin_1), J315.1 (Pin_1)
- net CS_U15: now also U301.18 (GPIO15)
- net CS_WING: now also J313.5 (Pin_5)
- net E5A: now also U409.3 (B); no longer U409.2 (A)
- net E5B: now also U409.2 (A); no longer U409.3 (B)
- net E6S: now also SW406.S1; no longer SW406.S2
- net E7A: now also U411.3 (B); no longer U411.2 (A)
- net E7B: now also U411.2 (A); no longer U411.3 (B)
- net EGND: now also SW406.S2, SW410.1 (GND), SW411.1 (GND), SW412.1 (GND), SW413.1 (GND), SW414.1 (GND), SW415.1 (GND), SW416.1 (GND), SW417.1 (GND), SW418.1 (GND), SW419.1 (GND); no longer SW406.S1
- net FGND: now also J309.6 (Pin_6), J313.1 (Pin_1); no longer J309.5 (Pin_5)
- net FSPI0MISO: now also J313.3 (Pin_3)
- net FSPI0MOSI: now also J313.6 (Pin_6)
- net FSPI0SCL: now also J313.4 (Pin_4)
- net FSPI1DC: now also J309.1 (Pin_1); no longer DS301.5 (RS), DS302.5 (RS), DS303.5 (RS), DS304.5 (RS), DS305.5 (RS)
- net FSPI1MISO: now also J309.2 (Pin_2); no longer J309.1 (Pin_1)
- net FSPI1MOSI: now also J309.3 (Pin_3); no longer DS301.3 (MOSI), DS302.3 (MOSI), DS303.3 (MOSI), DS304.3 (MOSI), DS305.3 (MOSI), J309.2 (Pin_2)
- net FSPI1SCL: now also J309.4 (Pin_4); no longer DS301.4 (SCK), DS302.4 (SCK), DS303.4 (SCK), DS304.4 (SCK), DS305.4 (SCK), J309.3 (Pin_3)
- net INT_OUT: now also J313.2 (Pin_2)
- net SPI1MOSI-ENC: now also DS301.3 (MOSI), DS302.3 (MOSI), DS303.3 (MOSI), DS304.3 (MOSI), DS305.3 (MOSI)
- net at SW302.2 (DIN): now also SW303.3 (DOUT)
- net at SW302.3 (DOUT): now also SW301.2 (DIN)
- net +B5V: now reaches SW302.4 (VCC)
- net +B5V: now also SW300.4 (VCC), SW301.4 (VCC), SW303.4 (VCC), SW304.4 (VCC), J314.3 (Pin_3), J315.3 (Pin_3)
- net at SW304.2 (DIN): now also J315.2 (Pin_2)
- net at SW304.3 (DOUT): now also SW303.2 (DIN)
- net +E5V: now reaches SW419.4 (VCC)
- net +E5V: now also SW410.4 (VCC), SW411.4 (VCC), SW412.4 (VCC), SW413.4 (VCC), SW414.4 (VCC), SW415.4 (VCC), SW416.4 (VCC), SW417.4 (VCC), SW418.4 (VCC)
- net at SW300.2 (DIN): now also SW301.3 (DOUT)
- net at SW300.3 (DOUT): now also J314.2 (Pin_2)
- new net SPI1DC-ENC: DS301.5 (RS), DS302.5 (RS), DS303.5 (RS), DS304.5 (RS), DS305.5 (RS), J310.6 (Pin_6)
- new net SPI1SCL-ENC: DS301.4 (SCK), DS302.4 (SCK), DS303.4 (SCK), DS304.4 (SCK), DS305.4 (SCK)
Other:
- note added: "SWAPPED!"
- note added: "TODO: rotate leds (swap 1/4 and 2/3 in symbol)"
- moved on the sheet: SW300, SW301, SW302, SW303, SW304
