File: kicad/Fader-Leds.kicad_sch (KiCad schematic)
At the start: 210 parts, among them U25 TLC59282, U26 TLC59282, U27 TLC59282, U28 TLC59282, U29 TLC59282, U30 TLC59282, U31 TLC59282, U32 TLC59282, U33 TLC59282, U34 TLC59282

Commit message: update kicad files
Parts:
- removed C80, C90: 100n, Capacitor_SMD:C_0603_1608Metric_Pad1.08x0.95mm_HandSolder, symbol Device:C
- removed D139, D156, D16, D164, D176, D178, D29, D36, D50, D82, D90, D99: LED, LED_SMD:LED_0603_1608Metric_Pad1.05x0.95mm_HandSolder, symbol Device:LED
- removed R46: 2K5, Resistor_SMD:R_0603_1608Metric_Pad0.98x0.95mm_HandSolder, symbol Device:R
Connections:
- net +E3V3: no longer C81.1, C82.1, C83.1, C84.1, D107.2 (A), D108.2 (A), D109.2 (A), D110.2 (A), D111.2 (A), D112.2 (A), D113.2 (A), D114.2 (A), D115.2 (A), D116.2 (A), D117.2 (A), D118.2 (A), D119.2 (A), D120.2 (A), D121.2 (A), D122.2 (A), D174.2 (A), U29.24 (VCC), U30.24 (VCC)
- net EGND: no longer C91.2, C92.2, R50.1, U31.1 (GND), U33.1 (GND)
- new net: C81.1, C82.1, U29.24 (VCC)
- new net: D107.2 (A), D108.2 (A), D109.2 (A), D110.2 (A), D111.2 (A), D112.2 (A), D113.2 (A), D114.2 (A), D115.2 (A), D116.2 (A), D117.2 (A), D118.2 (A), D119.2 (A), D120.2 (A), D121.2 (A), D122.2 (A), D174.2 (A)
- new net: C83.1, C84.1, U30.24 (VCC)
- new net: C91.2, C92.2

Commit message: changed some more of the schematic
Parts:
- added D139, D156, D16, D164, D176, D178, D29, D36, D50, D82, D90, D99: LED, LED_SMD:LED_0603_1608Metric_Pad1.05x0.95mm_HandSolder, symbol Device:LED
Connections:
- net +E3V3: now also D139.2 (A), D156.2 (A), D16.2 (A), D164.2 (A), D176.2 (A), D178.2 (A), D29.2 (A), D36.2 (A), D50.2 (A), D82.2 (A), D90.2 (A), D99.2 (A)
- net ENC0-5: now also D16.1 (K)
- net ENC1-2: now also D29.1 (K)
- net ENC1-9: now also D36.1 (K)
- net ENC2-7: now also D50.1 (K)
- net ENC4-15: now also D90.1 (K)
- net ENC4-7: now also D82.1 (K)
- net ENC5-8: now also D99.1 (K)
- net ENC7-DOT: now also D176.1 (K)
- net ENC8-0: now also D139.1 (K)
- net ENC8-DOT: now also D178.1 (K)
- net ENC9-1: now also D156.1 (K)
- net ENC9-9: now also D164.1 (K)

Commit message: continued work on fader pcb and redid all references more logicly
Parts:
- added C415, C425: 100n, Capacitor_SMD:C_0603_1608Metric_Pad1.08x0.95mm_HandSolder, symbol Device:C
- added R403: 2K5, Resistor_SMD:R_0603_1608Metric_Pad0.98x0.95mm_HandSolder, symbol Device:R
- renumbered C75 to C410, C76 to C411, C77 to C412, C78 to C413, C79 to C414, C81 to C416, C82 to C417, C83 to C418, C84 to C419, C85 to C420, C86 to C421, C87 to C422, C88 to C423, C89 to C424, C91 to C426, C92 to C427, D11 to D4000, D12 to D4001, D13 to D4002, D14 to D4003, D15 to D4004, D16 to D4005, D17 to D4006, D18 to D4007, D19 to D4008, D20 to D4009, D21 to D4010, D22 to D4011, D23 to D4012, D24 to D4013, D25 to D4014, D26 to D4015, D27 to D4016, D28 to D4017, D29 to D4018, D30 to D4019, D31 to D4020, D32 to D4021, D33 to D4022, D34 to D4023, D35 to D4024, D36 to D4025, D37 to D4026, D38 to D4027, D39 to D4028, D40 to D4029, D41 to D4030, D42 to D4031, D43 to D4032, D44 to D4033, D45 to D4034, D46 to D4035, D47 to D4036, D48 to D4037, D49 to D4038, D50 to D4039, D51 to D4040, D52 to D4041, D53 to D4042, D54 to D4043, D55 to D4044, D56 to D4045, D57 to D4046, D58 to D4047, D59 to D4048, D60 to D4049, D61 to D4050, D62 to D4051, D63 to D4052, D64 to D4053, D65 to D4054, D66 to D4055, D67 to D4056, D68 to D4057, D69 to D4058, D70 to D4059, D71 to D4060, D72 to D4061, D73 to D4062, D74 to D4063, D75 to D4064, D76 to D4065, D77 to D4066, D78 to D4067, D79 to D4068, D80 to D4069, D81 to D4070, D82 to D4071, D83 to D4072, D84 to D4073, D85 to D4074, D86 to D4075, D87 to D4076, D88 to D4077, D89 to D4078, D90 to D4079, D91 to D4080, D92 to D4081, D93 to D4082, D94 to D4083, D95 to D4084, D96 to D4085, D97 to D4086, D98 to D4087, D99 to D4088, D100 to D4089, D101 to D4090, D102 to D4091, D103 to D4092, D104 to D4093, D105 to D4094, D106 to D4095, D107 to D4096, D108 to D4097, D109 to D4098, D110 to D4099, D111 to D4100, D112 to D4101, D113 to D4102, D114 to D4103, D115 to D4104, D116 to D4105, D117 to D4106, D118 to D4107, D119 to D4108, D120 to D4109, D121 to D4110, D122 to D4111, D123 to D4112, D124 to D4113, D125 to D4114, D126 to D4115, D127 to D4116, D128 to D4117, D129 to D4118, D130 to D4119, D131 to D4120, D132 to D4121, D133 to D4122, D134 to D4123, D135 to D4124, D136 to D4125, D137 to D4126, D138 to D4127, D139 to D4128, D140 to D4129, D141 to D4130, D142 to D4131, D143 to D4132, D144 to D4133, D145 to D4134, D146 to D4135, D147 to D4136, D148 to D4137, D149 to D4138, D150 to D4139, D151 to D4140, D152 to D4141, D153 to D4142, D154 to D4143, D155 to D4144, D156 to D4145, D157 to D4146, D158 to D4147, D159 to D4148, D160 to D4149, D161 to D4150, D162 to D4151, D163 to D4152, D164 to D4153, D165 to D4154, D166 to D4155, D167 to D4156, D168 to D4157, D169 to D4158, D170 to D4159, D171 to D4160, D173 to D4161, D175 to D4162, D177 to D4163, D179 to D4164, D172 to D4165, D174 to D4166, D176 to D4167, D178 to D4168, D180 to D4169, R34 to R401, R35 to R402, R47 to R404, R48 to R405, R49 to R406, R50 to R407, R51 to R408, R52 to R409, R53 to R410, U25 to U414, U26 to U415, U27 to U416, U28 to U417, U29 to U418, U30 to U419, U31 to U420, U32 to U421, U33 to U422, U34 to U423
Connections:
- net +E3V3: now also C416.1, C417.1, C418.1, C419.1, U418.24 (VCC), U419.24 (VCC), C415.1, C425.1
- net EGND: now also R407.1, R408.1, U422.1 (GND), C415.2, C425.2, R403.1
- net at U416.23 (IREF): now also R403.2

Commit message: finish updateing all references, add schematic pdf and some more progress
Parts:
- renumbered C1 to C408, C2 to C409
Connections:
- net EGND: now also C426.2, C427.2, U420.1 (GND)
- net at U415.2 (SIN): now also U414.22 (SOUT)
- net at U415.22 (SOUT): now also U416.2 (SIN)
- net at U417.2 (SIN): now also U416.22 (SOUT)
- net at U417.22 (SOUT): now also U418.2 (SIN)
- net at U418.22 (SOUT): now also U419.2 (SIN)
- net at U421.2 (SIN): now also U420.22 (SOUT)
- net at U421.22 (SOUT): now also U422.2 (SIN)
- net at U423.2 (SIN): now also U422.22 (SOUT)
- net at U419.22 (SOUT): now also U420.2 (SIN)
Other:
- note added: "* 41.9"
- note added: "R_{IREF} (KΩ) ="
- note added: "V_{IREF} (V) ~{I_{OLC} (mA)}"
- note removed: "R_{IREF} (KΩ) = V_{IREF} (V) * 41.9 ~{I_{OLC} (mA)}"
- moved on the sheet: C408, C409, C410, C411, C412, C413, C414, C415, C416, C417, C418, C419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

Commit message: fix (schematic) : add missing power symbol to encoder leds
Connections:
- net +E3V3: now also D4096.2 (A), D4097.2 (A), D4098.2 (A), D4099.2 (A), D4100.2 (A), D4101.2 (A), D4102.2 (A), D4103.2 (A), D4104.2 (A), D4105.2 (A), D4106.2 (A), D4107.2 (A), D4108.2 (A), D4109.2 (A), D4110.2 (A), D4111.2 (A), D4166.2 (A)
Changed lines of the file:
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@@
+	)
+	(symbol
+		(lib_id "power:+3V3")
+		(at 303.53 279.4 0)
+		(unit 1)
+		(exclude_from_sim no)
+		(in_bom yes)
+		(on_board yes)
+		(dnp no)
+		(property "Reference" "#PWR05015"
+			(at 303.53 283.21 0)
+			(effects
+				(font
+					(size 1.27 1.27)
+				)
+				(hide yes)
+			)
+		)
+		(property "Value" "+E3V3"
+			(at 303.53 275.59 0)
+			(effects
+				(font
+					(size 1.27 1.27)
+				)
+			)
+		)
+		(property "Footprint" ""
+			(at 303.53 279.4 0)
+			(effects
+				(font
+					(size 1.27 1.27)
+				)
+				(hide yes)
+			)
+		)
+		(property "Datasheet" ""
+			(at 303.53 279.4 0)
+			(effects
+				(font
+					(size 1.27 1.27)
+				)
+				(hide yes)
+			)
+		)
+		(property "Description" ""
+			(at 303.53 279.4 0)
+			(effects
+				(font
+					(size 1.27 1.27)
+				)
+				(hide yes)
+			)
+		)
+		(pin "1"
+		)
+		(instances
+			(project "faders"
+				(path "/077511d1-9e66-4142-bbad-77a69cc748a7/a5bf4b9c-f855-46ea-be41-ff526471d004"
+					(reference "#PWR05015")
+					(unit 1)
+				)
+			)
+		)
 	)
 	(symbol
